Commit message: Add LiDAR sensor support to simulation
- Add lidar_link and lidar_joint to base_kinova_macro.xacro
- Add GPU LiDAR plugin to tidybot.gazebo.xacro
- Add lidar launch argument to launch_sim_robot.launch.py
- Add /scan and /scan/points topic bridges for ros_gz_bridge
- Update xacro parameter chain for lidar argument

Co-Authored-By: Claude Opus 4.6 <noreply@anthropic.com>

File: src/tidybot_description/urdf/base/tidybot++/base_kinova_macro.xacro (robot description, xacro)
@@ -2,5 +2,5 @@
 <robot name="tidybot_base" xmlns:xacro="http://ros.org/wiki/xacro">
     <xacro:property name="last_base_link" value="base"/>
-    <xacro:macro name="load_base" params="parent:='' prefix vision">
+    <xacro:macro name="load_base" params="parent:='' prefix vision lidar">
         <link name="world"></link>
         <link name="${prefix}base">
@@ -44,4 +44,32 @@
             </joint>
         </xacro:if>
+        <!-- LiDAR センサー -->
+        <link name="${prefix}lidar_link">
+            <inertial>
+                <origin xyz="0 0 0" rpy="0 0 0"/>
+                <mass value="0.1"/>
+                <inertia ixx="1e-6" ixy="0" ixz="0" iyy="1e-6" iyz="0" izz="1e-6"/>
+            </inertial>
+            <visual>
+                <origin xyz="0 0 0" rpy="0 0 0"/>
+                <geometry>
+                    <cylinder radius="0.035" length="0.04"/>
+                </geometry>
+                <material name="black">
+                    <color rgba="0.1 0.1 0.1 1"/>
+                </material>
+            </visual>
+            <collision>
+                <origin xyz="0 0 0" rpy="0 0 0"/>
+                <geometry>
+                    <cylinder radius="0.035" length="0.04"/>
+                </geometry>
+            </collision>
+        </link>
+        <joint name="${prefix}lidar_joint" type="fixed">
+            <origin xyz="0.3 0.0 0.15" rpy="0 0 0"/>
+            <parent link="${prefix}base"/>
+            <child link="${prefix}lidar_link"/>
+        </joint>
         <link name="joint_x_jointbody">
             <inertial>

File: src/tidybot_description/urdf/bot.xacro (robot description, xacro)
@@ -1,5 +1,5 @@
 <?xml version="1.0"?>
 <robot xmlns:xacro="http://ros.org/wiki/xacro">
-    <xacro:macro name="load_bot" params="arm gripper vision prefix">
+    <xacro:macro name="load_bot" params="arm gripper vision lidar prefix">
         <!-- load the corresponding macros -->
         <xacro:include filename="$(find tidybot_description)/urdf/arms/${arm}/${arm}_macro.xacro" />
@@ -7,5 +7,5 @@
         <xacro:include filename="$(find tidybot_description)/urdf/base/tidybot++/base_kinova_macro.xacro" />
         <!-- load the base -->
-        <xacro:load_base parent="" prefix="${prefix}" vision="${vision}" />
+        <xacro:load_base parent="" prefix="${prefix}" vision="${vision}" lidar="${lidar}" />
         <!-- load the arm -->
         <xacro:load_arm parent="${last_base_link}" vision="${vision}" prefix="${prefix}">

File: src/tidybot_description/urdf/tidybot.gazebo.xacro (robot description, xacro)
@@ -1,5 +1,5 @@
 <?xml version="1.0"?>
 <robot xmlns:xacro="http://ros.org/wiki/xacro">
-<xacro:macro name="load_gazebo_plugins" params="config_path prefix arm vision">
+<xacro:macro name="load_gazebo_plugins" params="config_path prefix arm vision lidar">
   <gazebo>
       <plugin name="gz_ros2_control::GazeboSimROS2ControlPlugin" filename="gz_ros2_control-system">
@@ -74,4 +74,34 @@
     </gazebo>
   </xacro:if>
+  <!-- GPU LiDAR プラグイン -->
+  <gazebo reference="${prefix}lidar_link">
+    <sensor name="${prefix}rplidar" type="gpu_lidar">
+      <always_on>1</always_on>
+      <update_rate>10</update_rate>
+      <visualize>true</visualize>
+      <topic>/scan</topic>
+      <gz_frame_id>${prefix}lidar_link</gz_frame_id>
+      <lidar>
+        <scan>
+          <horizontal>
+            <samples>360</samples>
+            <resolution>1.0</resolution>
+            <min_angle>-3.14159</min_angle>
+            <max_angle>3.14159</max_angle>
+          </horizontal>
+        </scan>
+        <range>
+          <min>0.15</min>
+          <max>12.0</max>
+          <resolution>0.015</resolution>
+        </range>
+        <noise>
+          <type>gaussian</type>
+          <mean>0.0</mean>
+          <stddev>0.01</stddev>
+        </noise>
+      </lidar>
+    </sensor>
+  </gazebo>
   <xacro:include filename="$(find tidybot_description)/urdf/arms/${arm}/${arm}_transmission.xacro" />
   <xacro:load_arm_transmission prefix="${prefix}" />

File: src/tidybot_description/urdf/tidybot.xacro (robot description, xacro)
@@ -8,9 +8,10 @@
     <xacro:arg name="base_mode" default="position" />
     <xacro:arg name="vision" default="true" />
+    <xacro:arg name="lidar" default="true" />
     <xacro:arg name="prefix" default="" />
     <xacro:arg name="ros2_control_config_path" default="$(find tidybot_description)/config/tidybot_controllers.yaml"/>
     <xacro:include filename="$(find tidybot_description)/urdf/bot.xacro" />
     <!-- load the robot -->
-    <xacro:load_bot arm="$(arg arm)" gripper="$(arg gripper)" vision="$(arg vision)" prefix="$(arg prefix)" />
+    <xacro:load_bot arm="$(arg arm)" gripper="$(arg gripper)" vision="$(arg vision)" lidar="$(arg lidar)" prefix="$(arg prefix)" />
     <!-- configure ros2_control joints -->
     <xacro:include filename="$(find tidybot_description)/urdf/tidybot.ros2_control.xacro" />
@@ -18,4 +19,4 @@
     <!-- load gazebo plugins -->
     <xacro:include filename="$(find tidybot_description)/urdf/tidybot.gazebo.xacro" />
-    <xacro:load_gazebo_plugins config_path="$(arg ros2_control_config_path)" prefix="$(arg prefix)" arm="$(arg arm)" vision="$(arg vision)" />
+    <xacro:load_gazebo_plugins config_path="$(arg ros2_control_config_path)" prefix="$(arg prefix)" arm="$(arg arm)" vision="$(arg vision)" lidar="$(arg lidar)" />
 </robot>
